Commit message: feat: SLAM working, map saved, TF relay, bridge config updated

File: config/robot.urdf.xacro (robot description, xacro)
@@ -7,7 +7,24 @@
   <xacro:a300 control="diff_4wd" front_wheels="outdoor" rear_wheels="outdoor"/>
   <!-- Attachments -->
+  <xacro:include filename="$(find clearpath_platform_description)/urdf/a300/attachments/bumper.urdf.xacro"/>
+  <xacro:bumper name="front_bumper" model="default" parent_link="front_bumper_mount" extension="0.0">
+    <origin xyz="0.0 0.0 0.0" rpy="0.0 0.0 0.0"/>
+  </xacro:bumper>
+  <xacro:include filename="$(find clearpath_platform_description)/urdf/a300/attachments/bumper.urdf.xacro"/>
+  <xacro:bumper name="rear_bumper" model="default" parent_link="rear_bumper_mount" extension="0.0">
+    <origin xyz="0.0 0.0 0.0" rpy="0.0 0.0 0.0"/>
+  </xacro:bumper>
+  <xacro:include filename="$(find clearpath_platform_description)/urdf/a300/attachments/top_plate.urdf.xacro"/>
+  <xacro:top_plate name="top_plate" model="default" parent_link="default_mount">
+    <origin xyz="0.0 0.0 0.0" rpy="0.0 0.0 0.0"/>
+  </xacro:top_plate>
   <!-- Links -->
   <!-- Mounts -->
   <!-- Sensors -->
+  <!-- lidar2d_0 -->
+  <xacro:include filename="$(find clearpath_sensors_description)/urdf/sick_lms1xx.urdf.xacro"/>
+  <xacro:sick_lms1xx name="lidar2d_0" parent_link="top_plate_front_mount" ang_res="0.5" min_ang="-2.391" max_ang="2.391" min_range="0.05" max_range="25.0" update_rate="40">
+    <origin xyz="0.0 0.0 0.0" rpy="0.0 0.0 0.0"/>
+  </xacro:sick_lms1xx>
   <!-- Manipulators -->
   <!-- Extras -->

Commit message: feat: Add camera to RViz, full task complete

File: config/robot.urdf.xacro (robot description, xacro)
@@ -27,4 +27,9 @@
     <origin xyz="0.0 0.0 0.0" rpy="0.0 0.0 0.0"/>
   </xacro:sick_lms1xx>
+  <!-- camera_0 -->
+  <xacro:include filename="$(find clearpath_sensors_description)/urdf/intel_realsense.urdf.xacro"/>
+  <xacro:intel_realsense name="camera_0" parent_link="top_plate_front_mount" update_rate="30" image_height="480" image_width="640" model="d435">
+    <origin xyz="0.1 0.0 0.1" rpy="0.0 0.0 0.0"/>
+  </xacro:intel_realsense>
   <!-- Manipulators -->
   <!-- Extras -->
